File: HARDWARE/TWERCC.sch (EAGLE design)
At the start: 28 parts, among them U1 MSP430F5342_RGZ_48

Commit message: Altered Name
Other:
- note added: "TWERCC"
- moved on the sheet: C10, C11, C9, D1, D2, D3, JP1, JP2, JP3, R1, R2, R3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
